File: eagle/sword.brd (EAGLE design)
At the start: 20 x 54 mm, 6 parts, among them U1 TINY45-20-DIP

Commit message: shrunk just a little
Parts:
- moved S1 2.54 mm to (9.84, 42.5)
- moved J1 1.27 mm to (3.81, 25.4)
- moved U1 1.27 mm to (10.2, 31.8)
- moved J4 1.27 mm to (6.35, 7.62)
- moved J3 1.27 mm to (14.0, 2.54)
- moved J2 1.27 mm to (11.4, 20.3)
Routing:
- net DIN: track 17.0 -> 13.2 mm
- net N$1: track 32.3 -> 28.5 mm
- net GND: track 38.5 -> 34.7 mm
- net VCC: track 6.00 -> 4.73 mm
Other:
- board size 20 x 54 mm -> 20 x 48.9 mm
Changed lines of the file:
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@@
 <setting verticaltext="up"/>
 </settings>
-<grid distance="0.1" unitdist="inch" unit="inch" style="lines" multiple="1" display="no" altdistance="0.025" altunitdist="inch" altunit="inch"/>
+<grid distance="0.05" unitdist="inch" unit="inch" style="lines" multiple="1" display="no" altdistance="0.025" altunitdist="inch" altunit="inch"/>
 <layers>
 <layer number="1" name="Top" color="4" fill="1" visible="yes" active="yes"/>
@@
 <plain>
 <wire x1="0" y1="0" x2="19.99" y2="0" width="0" layer="20"/>
-<wire x1="19.99" y1="0" x2="19.99" y2="53.965" width="0" layer="20"/>
-<wire x1="19.99" y1="53.965" x2="0" y2="53.965" width="0" layer="20"/>
-<wire x1="0" y1="53.965" x2="0" y2="0" width="0" layer="20"/>
+<wire x1="19.99" y1="0" x2="19.99" y2="48.885" width="0" layer="20"/>
+<wire x1="19.99" y1="48.885" x2="0" y2="48.885" width="0" layer="20"/>
+<wire x1="0" y1="48.885" x2="0" y2="0" width="0" layer="20"/>
 </plain>
 <attributes>
@@
 </autorouter>
 <elements>
-<element name="J1" library="SparkFun-Connectors" package="1X01_LONGPAD" value="" x="3.81" y="26.67" rot="R270"/>
-<element name="J2" library="SparkFun-Connectors" package="1X01_LONGPAD" value="" x="11.43" y="21.59" rot="R90"/>
-<element name="S1" library="switch-omron" package="B3F-10XX" value="" x="9.8425" y="45.085" rot="R180">
-<attribute name="OC_NEWARK" value="36M3542" x="9.8425" y="45.085" size="1.778" layer="27" rot="R180" display="off"/>
-<attribute name="MF" value="" x="9.8425" y="45.085" size="1.778" layer="27" rot="R180" display="off"/>
-<attribute name="MPN" value="B3F-1000" x="9.8425" y="45.085" size="1.778" layer="27" rot="R180" display="off"/>
-<attribute name="OC_FARNELL" value="176432" x="9.8425" y="45.085" size="1.778" layer="27" rot="R180" display="off"/>
+<element name="J1" library="SparkFun-Connectors" package="1X01_LONGPAD" value="" x="3.81" y="25.4" rot="R270"/>
+<element name="J2" library="SparkFun-Connectors" package="1X01_LONGPAD" value="" x="11.43" y="20.32" rot="R90"/>
+<element name="S1" library="switch-omron" package="B3F-10XX" value="" x="9.8425" y="42.545" rot="R180">
+<attribute name="OC_NEWARK" value="36M3542" x="9.8425" y="42.545" size="1.778" layer="27" rot="R180" display="off"/>
+<attribute name="MF" value="" x="9.8425" y="42.545" size="1.778" layer="27" rot="R180" display="off"/>
+<attribute name="MPN" value="B3F-1000" x="9.8425" y="42.545" size="1.778" layer="27" rot="R180" display="off"/>
+<attribute name="OC_FARNELL" value="176432" x="9.8425" y="42.545" size="1.778" layer="27" rot="R180" display="off"/>
 </element>
-<element name="U1" library="SparkFun-DigitalIC" package="DIP08" value="TINY45-20-DIP" x="10.16" y="33.02">
-<attribute name="PROD_ID" value="IC-09439" x="10.16" y="33.02" size="1.778" layer="27" display="off"/>
+<element name="U1" library="SparkFun-DigitalIC" package="DIP08" value="TINY45-20-DIP" x="10.16" y="31.75">
+<attribute name="PROD_ID" value="IC-09439" x="10.16" y="31.75" size="1.778" layer="27" display="off"/>
 </element>
-<element name="J3" library="SparkFun-Connectors" package="1X01_LONGPAD" value="" x="13.97" y="3.81" rot="R90"/>
-<element name="J4" library="SparkFun-Connectors" package="1X01_LONGPAD" value="" x="6.35" y="8.89" rot="R90"/>
+<element name="J3" library="SparkFun-Connectors" package="1X01_LONGPAD" value="" x="13.97" y="2.54" rot="R90"/>
+<element name="J4" library="SparkFun-Connectors" package="1X01_LONGPAD" value="" x="6.35" y="7.62" rot="R90"/>
 </elements>
 <signals>
@@
 <contactref element="U1" pad="8"/>
 <contactref element="S1" pad="2"/>
-<wire x1="6.35" y1="36.83" x2="6.5913" y2="42.8244" width="0.8128" layer="16"/>
+<wire x1="6.35" y1="35.56" x2="6.5913" y2="40.2844" width="0.8128" layer="16"/>
 </signal>
 <signal name="GND">
@@
 <contactref element="J2" pad="1"/>
 <polygon width="1.27" layer="16" thermals="no">
-<vertex x="-0.635" y="53.975"/>
-<vertex x="20.955" y="53.975"/>
+<vertex x="-0.635" y="48.895"/>
+<vertex x="20.955" y="48.895"/>
 <vertex x="21.59" y="-0.635"/>
 <vertex x="-0.635" y="-0.635"/>
 </polygon>
-<wire x1="11.43" y1="21.59" x2="15.875" y2="26.67" width="0.8128" layer="16"/>
-<wire x1="15.875" y1="26.67" x2="15.875" y2="49.53" width="0.8128" layer="16"/>
-<wire x1="15.875" y1="49.53" x2="11.1125" y2="49.53" width="0.8128" layer="16"/>
-<wire x1="11.1125" y1="49.53" x2="11.1125" y2="53.6575" width="0.8128" layer="16"/>
-<wire x1="11.43" y1="21.59" x2="13.97" y2="29.21" width="0" layer="19" extent="1-1"/>
+<wire x1="11.43" y1="20.32" x2="15.875" y2="25.4" width="0.8128" layer="16"/>
+<wire x1="15.875" y1="25.4" x2="15.875" y2="46.99" width="0.8128" layer="16"/>
+<wire x1="15.875" y1="46.99" x2="11.1125" y2="46.99" width="0.8128" layer="16"/>
+<wire x1="11.1125" y1="46.99" x2="11.1125" y2="48.5775" width="0.8128" layer="16"/>
+<wire x1="11.43" y1="20.32" x2="13.97" y2="27.94" width="0" layer="19" extent="1-1"/>
 </signal>
 <signal name="DIN">
 <contactref element="U1" pad="7"/>
-<wire x1="8.89" y1="36.83" x2="9.8425" y2="39.0525" width="0.8128" layer="16"/>
-<wire x1="9.8425" y1="39.0525" x2="9.8425" y2="53.6575" width="0.8128" layer="16"/>
+<wire x1="8.89" y1="35.56" x2="9.8425" y2="37.7825" width="0.8128" layer="16"/>
+<wire x1="9.8425" y1="37.7825" x2="9.8425" y2="48.5775" width="0.8128" layer="16"/>
 </signal>
 <signal name="N$1">
 <contactref element="J1" pad="1"/>
 <contactref element="S1" pad="4"/>
-<wire x1="3.81" y1="26.67" x2="4.1275" y2="26.67" width="0.8128" layer="16"/>
-<wire x1="4.1275" y1="26.67" x2="4.1275" y2="47.625" width="0.8128" layer="16"/>
-<wire x1="4.1275" y1="47.625" x2="6.5913" y2="47.625" width="0.8128" layer="16"/>
-<wire x1="6.5913" y1="47.625" x2="6.5913" y2="47.3456" width="0.8128" layer="16"/>
-<wire x1="6.5913" y1="47.3456" x2="8.5725" y2="47.3456" width="0.8128" layer="16"/>
-<wire x1="8.5725" y1="47.3456" x2="8.5725" y2="53.6575" width="0.8128" layer="16"/>
+<wire x1="3.81" y1="25.4" x2="4.1275" y2="25.4" width="0.8128" layer="16"/>
+<wire x1="4.1275" y1="25.4" x2="4.1275" y2="45.085" width="0.8128" layer="16"/>
+<wire x1="4.1275" y1="45.085" x2="6.5913" y2="45.085" width="0.8128" layer="16"/>
+<wire x1="6.5913" y1="45.085" x2="6.5913" y2="44.8056" width="0.8128" layer="16"/>
+<wire x1="6.5913" y1="44.8056" x2="8.5725" y2="44.8056" width="0.8128" layer="16"/>
+<wire x1="8.5725" y1="44.8056" x2="8.5725" y2="48.5775" width="0.8128" layer="16"/>
 </signal>
 </signals>

Commit message: changed board to use a standard cr2032 socket
Parts:
- removed J3, J4: (no value), SparkFun-Connectors:1X01_LONGPAD
- added PAD1: NEO_VCC, wirepad:SMD1,27-2,54
- added PAD2: NEO_DIN, wirepad:SMD1,27-2,54
- added PAD3: NEO_GND, wirepad:SMD1,27-2,54
- J1: value (none) -> VCC_IN
- J2: value (none) -> GND
- S1: value (none) -> PWR_SW
- moved J2 23.0 mm to (26.0, 2.54)
- moved J1 22.9 mm to (3.17, 2.54)
- moved S1 11.8 mm to (15.9, 32.4)
- moved U1 11.7 mm to (15.9, 21.6)
Connections:
- net N$1 renamed VCC_SW
- net DIN: now also PAD2.1
- net GND: now also PAD3.1
- net VCC: now also PAD1.1
Routing:
- net GND: track 34.7 -> 0.00 mm
- net VCC: track 4.73 -> 15.7 mm
- net VCC_SW: track 28.5 -> 37.0 mm
- net DIN: track 13.2 -> 14.4 mm
Other:
- board size 20 x 48.9 mm -> 31.8 x 40.6 mm
Changed lines of the file:
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@@
 <setting verticaltext="up"/>
 </settings>
-<grid distance="0.05" unitdist="inch" unit="inch" style="lines" multiple="1" display="no" altdistance="0.025" altunitdist="inch" altunit="inch"/>
+<grid distance="0.0125" unitdist="inch" unit="inch" style="lines" multiple="1" display="no" altdistance="0.025" altunitdist="inch" altunit="inch"/>
 <layers>
 <layer number="1" name="Top" color="4" fill="1" visible="yes" active="yes"/>
@@
 <board>
 <plain>
-<wire x1="0" y1="0" x2="19.99" y2="0" width="0" layer="20"/>
-<wire x1="19.99" y1="0" x2="19.99" y2="48.885" width="0" layer="20"/>
-<wire x1="19.99" y1="48.885" x2="0" y2="48.885" width="0" layer="20"/>
-<wire x1="0" y1="48.885" x2="0" y2="0" width="0" layer="20"/>
+<wire x1="0" y1="0" x2="31.75" y2="0" width="0" layer="20"/>
+<wire x1="31.75" y1="0" x2="31.75" y2="40.64" width="0" layer="20"/>
+<wire x1="31.75" y1="40.64" x2="0" y2="40.64" width="0" layer="20"/>
+<wire x1="0" y1="40.64" x2="0" y2="0" width="0" layer="20"/>
 </plain>
 <attributes>
@@
 </autorouter>
 <elements>
-<element name="J1" library="SparkFun-Connectors" package="1X01_LONGPAD" value="" x="3.81" y="25.4" rot="R270"/>
-<element name="J2" library="SparkFun-Connectors" package="1X01_LONGPAD" value="" x="11.43" y="20.32" rot="R90"/>
-<element name="S1" library="switch-omron" package="B3F-10XX" value="" x="9.8425" y="42.545" rot="R180">
-<attribute name="OC_NEWARK" value="36M3542" x="9.8425" y="42.545" size="1.778" layer="27" rot="R180" display="off"/>
-<attribute name="MF" value="" x="9.8425" y="42.545" size="1.778" layer="27" rot="R180" display="off"/>
-<attribute name="MPN" value="B3F-1000" x="9.8425" y="42.545" size="1.778" layer="27" rot="R180" display="off"/>
-<attribute name="OC_FARNELL" value="176432" x="9.8425" y="42.545" size="1.778" layer="27" rot="R180" display="off"/>
-</element>
-<element name="U1" library="SparkFun-DigitalIC" package="DIP08" value="TINY45-20-DIP" x="10.16" y="31.75">
-<attribute name="PROD_ID" value="IC-09439" x="10.16" y="31.75" size="1.778" layer="27" display="off"/>
-</element>
-<element name="J3" library="SparkFun-Connectors" package="1X01_LONGPAD" value="" x="13.97" y="2.54" rot="R90"/>
-<element name="J4" library="SparkFun-Connectors" package="1X01_LONGPAD" value="" x="6.35" y="7.62" rot="R90"/>
+<element name="J1" library="SparkFun-Connectors" package="1X01_LONGPAD" value="VCC_IN" x="3.175" y="2.54" smashed="yes" rot="R270"/>
+<element name="J2" library="SparkFun-Connectors" package="1X01_LONGPAD" value="GND" x="26.035" y="2.54" smashed="yes" rot="R90"/>
+<element name="S1" library="switch-omron" package="B3F-10XX" value="PWR_SW" x="15.875" y="32.385" smashed="yes" rot="R180">
+<attribute name="OC_NEWARK" value="36M3542" x="15.875" y="32.385" size="1.778" layer="27" rot="R180" display="off"/>
+<attribute name="MF" value="" x="15.875" y="32.385" size="1.778" layer="27" rot="R180" display="off"/>
+<attribute name="MPN" value="B3F-1000" x="15.875" y="32.385" size="1.778" layer="27" rot="R180" display="off"/>
+<attribute name="OC_FARNELL" value="176432" x="15.875" y="32.385" size="1.778" layer="27" rot="R180" display="off"/>
+</element>
+<element name="U1" library="SparkFun-DigitalIC" package="DIP08" value="TINY45-20-DIP" x="15.875" y="21.59" smashed="yes">
+<attribute name="PROD_ID" value="IC-09439" x="15.875" y="21.59" size="1.778" layer="27" display="off"/>
+</element>
+<element name="PAD1" library="wirepad" package="SMD1,27-2,54" value="NEO_VCC" x="13.335" y="39.37" smashed="yes" rot="MR0">
+<attribute name="VALUE" x="13.335" y="39.37" size="0.0254" layer="28" rot="MR0"/>
+</element>
+<element name="PAD2" library="wirepad" package="SMD1,27-2,54" value="NEO_DIN" x="15.875" y="39.37" smashed="yes" rot="MR0">
+<attribute name="VALUE" x="15.875" y="39.37" size="0.0254" layer="28" rot="MR0"/>
+</element>
+<element name="PAD3" library="wirepad" package="SMD1,27-2,54" value="NEO_GND" x="18.415" y="39.37" smashed="yes" rot="MR0">
+<attribute name="VALUE" x="18.415" y="39.37" size="0.0254" layer="28" rot="MR0"/>
+</element>
 </elements>
 <signals>
@@
 <contactref element="U1" pad="8"/>
 <contactref element="S1" pad="2"/>
-<wire x1="6.35" y1="35.56" x2="6.5913" y2="40.2844" width="0.8128" layer="16"/>
+<wire x1="12.6238" y1="30.1244" x2="12.065" y2="25.4" width="0.8128" layer="16"/>
+<contactref element="PAD1" pad="1"/>
+<wire x1="13.335" y1="39.37" x2="13.335" y2="36.83" width="0.8128" layer="16"/>
+<wire x1="13.335" y1="36.83" x2="14.605" y2="36.5125" width="0.8128" layer="16"/>
+<wire x1="14.605" y1="36.5125" x2="14.9225" y2="33.655" width="0.8128" layer="16"/>
+<wire x1="14.9225" y1="33.655" x2="12.6238" y2="30.1244" width="0.8128" layer="16"/>
 </signal>
 <signal name="GND">
@@
 <contactref element="J2" pad="1"/>
 <polygon width="1.27" layer="16" thermals="no">
-<vertex x="-0.635" y="48.895"/>
-<vertex x="20.955" y="48.895"/>
-<vertex x="21.59" y="-0.635"/>
-<vertex x="-0.635" y="-0.635"/>
+<vertex x="-2.54" y="41.91"/>
+<vertex x="34.29" y="41.91"/>
+<vertex x="34.29" y="-2.54"/>
+<vertex x="-2.54" y="-2.54"/>
 </polygon>
-<wire x1="11.43" y1="20.32" x2="15.875" y2="25.4" width="0.8128" layer="16"/>
-<wire x1="15.875" y1="25.4" x2="15.875" y2="46.99" width="0.8128" layer="16"/>
-<wire x1="15.875" y1="46.99" x2="11.1125" y2="46.99" width="0.8128" layer="16"/>
-<wire x1="11.1125" y1="46.99" x2="11.1125" y2="48.5775" width="0.8128" layer="16"/>
-<wire x1="11.43" y1="20.32" x2="13.97" y2="27.94" width="0" layer="19" extent="1-1"/>
+<contactref element="PAD3" pad="1"/>
 </signal>
 <signal name="DIN">
 <contactref element="U1" pad="7"/>
-<wire x1="8.89" y1="35.56" x2="9.8425" y2="37.7825" width="0.8128" layer="16"/>
-<wire x1="9.8425" y1="37.7825" x2="9.8425" y2="48.5775" width="0.8128" layer="16"/>
+<contactref element="PAD2" pad="1"/>
+<wire x1="15.5575" y1="28.575" x2="14.605" y2="25.4" width="0.8128" layer="16"/>
+<wire x1="15.875" y1="39.37" x2="16.1925" y2="36.83" width="0.8128" layer="16"/>
+<wire x1="16.1925" y1="36.83" x2="16.8275" y2="33.3375" width="0.8128" layer="16"/>
+<wire x1="16.8275" y1="33.3375" x2="15.5575" y2="28.575" width="0.8128" layer="16"/>
 </signal>
-<signal name="N$1">
+<signal name="VCC_SW">
 <contactref element="J1" pad="1"/>
 <contactref element="S1" pad="4"/>
-<wire x1="3.81" y1="25.4" x2="4.1275" y2="25.4" width="0.8128" layer="16"/>
-<wire x1="4.1275" y1="25.4" x2="4.1275" y2="45.085" width="0.8128" layer="16"/>
-<wire x1="4.1275" y1="45.085" x2="6.5913" y2="45.085" width="0.8128" layer="16"/>
-<wire x1="6.5913" y1="45.085" x2="6.5913" y2="44.8056" width="0.8128" layer="16"/>
-<wire x1="6.5913" y1="44.8056" x2="8.5725" y2="44.8056" width="0.8128" layer="16"/>
-<wire x1="8.5725" y1="44.8056" x2="8.5725" y2="48.5775" width="0.8128" layer="16"/>
+<wire x1="12.6238" y1="34.6456" x2="3.175" y2="28.0543" width="0.8128" layer="16"/>
+<wire x1="3.175" y1="28.0543" x2="3.175" y2="2.54" width="0.8128" layer="16"/>
 </signal>
 </signals>
